Commit message: Fix orbbec astra frames

File: urdf/calibration/extrinsic_camera_calibration_constants.urdf.xacro (robot description, xacro)
@@ -12,8 +12,8 @@
 <xacro:macro name="camera_baseline_constants" params="camera_model" >
   <xacro:if value="${camera_model == 'orbbec-astra'}">
-    <origin xyz="0.0 0.047 0.0" rpy="0 0 0" />
+    <origin xyz="-0.0006 0.0375 -0.015" rpy="0 0 0" />
   </xacro:if>
   <xacro:if value="${camera_model == 'orbbec-astra-pro'}">
-    <origin xyz="0.0 0.047 0.0" rpy="0 0 0" />
+    <origin xyz="-0.0006 0.0375 -0.015" rpy="0 0 0" />
   </xacro:if>
   <xacro:if value="${camera_model == 'asus-xtion'}">
